File: pcb/data_logger/data_logger.kicad_sch (KiCad schematic)
At the start: 2 parts, among them U1 ESP32-WROOM-32, U2 AMS1117

Commit message: alles sauber
Parts:
- removed U1: ESP32-WROOM-32, RF_Module:ESP32-WROOM-32, symbol RF_Module:ESP32-WROOM-32
- removed U2: AMS1117, PCM_JLCPCB:SOT-223-3_L6.5-W3.4-P2.30-LS7.0-BR, symbol PCM_JLCPCB-Power:LDO, 3.3V, 1A
- added C1: 10uF, C10uF:CAPC1005X70N, symbol C10uF:GRT155R60J106ME13J
- added C10, C9: C10uF, C10uF:CAPC1005X70N, symbol C10uF:GRT155R60J106ME13J
- added C11, C8: 01.uF, C0.1uF:CAPC2012X94N, symbol C0.1uF:08055C104KAT2A
- added C12: C4.7uF, C4.7uF:C0805, symbol C4.7uF:C0805C475K4RACAUTO
- added C13: C2.2uF, C2.2uF:CAPC2012X145N, symbol C2.2uF:C2012X7R2A225K125AC
- added C2, C3: 08055C104KAT2A, C0.1uF:CAPC2012X94N, symbol C0.1uF:08055C104KAT2A
- added C4, C5: 1uF, C1uF:CAPC2012X140N, symbol C1uF:KAF21KR71H105KU
- added C6, C7: 0.1uF, C0.1uF:CAPC2012X94N, symbol C0.1uF:08055C104KAT2A
- added D1: 3A-10V-280mV, D-3A-10V-300mV:SOD2513X110N, symbol D-3A-10V-280mV:BAT60AE6327HTSA1
- added H1, H2, H3, H4: MountingHole_Pad, MountingHole:MountingHole_3.2mm_M3_DIN965_Pad_TopBottom, symbol Mechanical:MountingHole_Pad
- added HM1: BME280, BME280:BME280, symbol BME280:BME280
- added IC1: ESP32-S3-WROOM-2-N32R8V, ESP32-S3-WROOM-2:ESP32S3WROOM2N32R8V, symbol ESP32-S3-WROOM-2-N32R8V:ESP32-S3-WROOM-2-N32R8V
- added IC2: MBT3904DW1T1G, MBT3904DW1T1G:SOT65P210X110-6N, symbol MBT3904DW1T1G:MBT3904DW1T1G
- added IC3: MAX17048G+T10, sparkfun_import:DFN-8, symbol MAX17048G+T10:MAX17048G+T10
- added IC4: MIC94310-GYMT-TR, MIC94310-GYMT-TR:SON50P155X120X60-5N-D, symbol MIC94310-GYMT-TR:MIC94310-GYMT-TR
- added IC5: TXS0108EQPWRQ1, TXS0108E:SOP65P640X120-20N, symbol TXS0108EQPWRQ1:TXS0108EQPWRQ1
- added IC6: AP2112K-3.3TRG1, AP2112K-3.3V:SOT95P282X130-5N, symbol AP2112K-3_3TRG1:AP2112K-3.3TRG1
- added IC7: ICM-20948, ICM-20948:QFN40P300X300X105-25N-D, symbol ICM-20948:ICM-20948
- added IC8: MCP73831T-2ACI_OT, MCP73831:SOT95P270X145-5N, symbol MCP73831T-2ACI_OT:MCP73831T-2ACI_OT
- added J1: UJ32-C-H-G-H2-SMT-TR, USB-C:UJ32CHGH2SMTTR, symbol USB-C:UJ32-C-H-G-H2-SMT-TR
- added J10: TXS0108E, Jumper:SolderJumper-2_P1.3mm_Open_RoundedPad1.0x1.5mm, symbol Connector:Conn_01x02_Pin
- added J11: 1769, Connector_JST:JST_EH_S2B-EH_1x02_P2.50mm_Horizontal, symbol JST:1769
- added J12: ~, Jumper:SolderJumper-3_P1.3mm_Open_RoundedPad1.0x1.5mm, symbol Connector:Conn_01x03_Pin
- added J2: 045138008100858+, SD-Card-Slot-2:045138008100858, symbol SD-Card-Slot-2:045138008100858+
- added J3, J4: Conn_01x20_Pin, Connector_PinSocket_2.54mm:PinSocket_1x20_P2.54mm_Vertical, symbol Connector:Conn_01x20_Pin
- added J5, J7: Conn_01x04, Connector_PinSocket_2.54mm:PinSocket_1x04_P2.54mm_Vertical, symbol Connector_Generic:Conn_01x04
- added J6: Conn_01x03_Pin, Jumper:SolderJumper-3_P1.3mm_Open_RoundedPad1.0x1.5mm_NumberLabels, symbol Connector:Conn_01x03_Pin
- added J8: Conn_01x04, Connector_JST:JST_SH_BM04B-SRSS-TB_1x04-1MP_P1.00mm_Vertical, symbol Connector_Generic:Conn_01x04
- added J9: LiPo, Jumper:SolderJumper-2_P1.3mm_Bridged_RoundedPad1.0x1.5mm, symbol Connector:Conn_01x02_Pin
- added LED1: VLMY234ABCA-GS08, LED-yellow:LEDM2214X140N, symbol LED-yellow:VLMY234ABCA-GS08
- added PowerLED1, PowerLED2: 150080RS75000, LED-red:LEDC2012X80N, symbol LED-red:150080RS75000
- added R1, R2: 5.1k, R5.1k:RESC3116X65N, symbol R5.1k:CHP1206AFX-5101ELF
- added R10, R11, R12, R15, R7, R9: R0, R0:RESC2013X84N, symbol R0:WSL080500000ZEA9
- added R13, R14, R16: MCU0805MD1000BP100, RESC2012X62N, symbol R100:MCU0805MD1000BP100
- added R17, R18: 330k, R330k:RESC2012X50N, symbol R330k:RCV0805330KJNEA
- added R19: R2.2k, R2.2k:RESC2013X65N, symbol R2.2k:TNPW08052K20BEEA
- added R20, R21, R22, R5, R6, R8: R4.7k, R4.7k:RESC2012X50N, symbol R4.7k:CRCW08054K70FKEC
- added R3, R4: 10k, R10k:RESC1608X55N, symbol R10k:MCT0603MG1002BP500
- added U1: CH340C, Package_SO:SOIC-16_3.9x9.9mm_P1.27mm, symbol Interface_USB:CH340C
Connections:
- net +3V3: now also C1.2, C13.2, C2.2, C5.2, C6.2, C7.2, C8.2, C9.2, HM1.6 (VDDIO), HM1.8 (VDD), IC1.2 (3V3), IC4.4 (VIN), IC5.19 (VCCB), IC6.5 (VOUT), J2.4 (VDD), J4.18 (Pin_18), J7.1 (Pin_1), J8.3 (Pin_3), PowerLED1.2 (A), R21.2, R22.2, R5.2, R6.2, R8.2, U1.16 (VCC), U1.4 (V3)
- net +5V: now also IC6.1 (VIN), J1.A4 (VBUS_1), J1.A9 (VBUS_2), J1.B4 (VBUS_3), J1.B9 (VBUS_4), J4.19 (Pin_19), J5.1 (Pin_1), J9.1 (Pin_1), R17.2
- net GND: now also C1.1, C10.1, C11.1, C12.1, C13.1, C2.1, C3.1, C4.1, C5.1, C6.1, C7.1, C8.1, C9.1, H1.1, H2.1, H3.1, H4.1, HM1.1 (GND_1), HM1.7 (GND_2), IC1.1 (GND_1), IC1.40 (GND_2), IC1.41 (GND_3), IC1.42 (GND_4), IC1.43 (GND_5), IC1.44 (GND_6), IC1.45 (GND_7), IC1.46 (GND_8), IC1.47 (GND_9), IC1.48 (GND_10), IC1.49 (GND_11), IC3.1 (CTG), IC3.4 (GND), IC3.6 (QSTRT), IC4.2 (GND), IC5.11 (GND), IC6.2 (GND), IC7.18 (GND), IC8.2 (VSS), J1.A1 (GND_1), J1.A12 (GND_2), J1.B1 (GND_3), J1.B12 (GND_4), J1.MH1, J1.MH2, J1.MP1, J1.MP2, J11.1, J12.3 (Pin_3), J2.10, J2.11, J2.12, J2.13, J2.6 (VSS), J4.1 (Pin_1), J4.20 (Pin_20), J5.4 (Pin_4), J6.3 (Pin_3), J7.4 (Pin_4), J8.4 (Pin_4), R1.1, R13.2, R14.2, R18.1, R19.1, R2.1, U1.1 (GND)
- new net: J12.1 (Pin_1), R20.1
- new net: IC7.9 (SDO_/_AD0), J12.2 (Pin_2)
- new net: J1.B5 (CC2), R1.2
- new net: IC2.2 (B_2), R3.2
- new net: IC2.5 (B_1), R4.1
- new net: R7.1, U1.2 (TXD)
- new net: IC4.3 (EN), R8.1
- new net: HM1.2 (CSB), R6.1
- new net: IC8.1 (STAT), R16.2
- new net: D1.1 (K), IC8.4 (VDD), J9.2 (Pin_2), LED1.2 (A)
- new net: IC8.5 (PROG), R19.2
- new net: HM1.5 (SDO), J6.2 (Pin_2)
- new net: J6.1 (Pin_1), R5.1
- new net: PowerLED2.1 (K), R14.1
- new net: R12.2, R15.2, U1.6 (UD-)
- new net: IC6.3 (EN), R17.1
- new net: PowerLED1.1 (K), R13.1
- new net: IC5.10 (OE), J10.2 (Pin_2), R18.2
- new net: R11.2, R9.2, U1.5 (UD+)
- new net: LED1.1 (K), R16.1
- new net: J1.A5 (CC1), R2.2
- new net: R10.1, U1.3 (RXD)
- new net +1V8: C10.2, C11.2, C4.2, IC4.1 (VOUT), IC5.2 (VCCA), IC7.13 (VDD), IC7.8 (VDDIO), J10.1 (Pin_1), J4.3 (Pin_3), R20.2
- new net +3V8: C12.2, C3.2, D1.2 (A), IC3.2 (CELL), IC3.3 (VDD), IC8.3 (VBAT), J11.2, J4.2 (Pin_2)
- new net CH340_DTR: IC2.4 (E_1), R4.2, U1.13 (~{DTR})
- new net CH340_RTS: IC2.1 (E_2), R3.1, U1.14 (~{RTS})
- new net CHIP_BOOT: IC1.27 (IO0), IC2.6 (C_2), J4.13 (Pin_13)
- new net CHIP_RX: IC1.36 (RXD0), J4.7 (Pin_7), J7.2 (Pin_2), R7.2
- new net CHIP_TX: IC1.37 (TXD0), J4.6 (Pin_6), J7.3 (Pin_3), R10.2
- new net Chip_EN: IC1.3 (EN), IC2.3 (C_1), J3.1 (Pin_1)
- new net DN1: J1.A7 (DN1), J5.3 (Pin_3), R12.1
- new net DN2: J1.B7 (DN2), R15.1
- new net DP1: J1.A6 (DP1), J5.2 (Pin_2), R9.1
- new net DP2: J1.B6 (DP2), R11.1
- new net GPIO1: IC1.39 (IO1), J4.4 (Pin_4)
- new net GPIO10: IC1.18 (IO10), J3.16 (Pin_16), PowerLED2.2 (A)
- new net GPIO11: IC1.19 (IO11), J3.17 (Pin_17)
- new net GPIO12: IC1.20 (IO12), J3.18 (Pin_18)
- new net GPIO13: IC1.21 (IO13), J3.19 (Pin_19)
- new net GPIO14: IC1.22 (IO14), J3.20 (Pin_20)
- new net GPIO15: IC1.8 (IO15), J3.6 (Pin_6)
- new net GPIO18_CLK: IC1.11 (IO18), J2.5 (CLK), J3.9 (Pin_9)
- new net GPIO19_MISO: IC1.13 (IO19), J2.7 (DAT0), J3.11 (Pin_11)
- new net GPIO2: IC1.38 (IO2), J4.5 (Pin_5)
- new net GPIO20_MOSI: IC1.14 (IO20), J2.3 (CMD), J3.12 (Pin_12)
- new net GPIO21: IC1.23 (IO21), J4.17 (Pin_17)
- new net GPIO3: IC1.15 (IO3), J3.13 (Pin_13)
- new net GPIO38: IC1.31 (IO38), J4.12 (Pin_12)
- new net GPIO39: IC1.32 (IO39), J4.11 (Pin_11)
- new net GPIO4: IC1.4 (IO4), J3.2 (Pin_2)
- new net GPIO40: IC1.33 (IO40), J4.10 (Pin_10)
- new net GPIO41: IC1.34 (IO41), J4.9 (Pin_9)
- new net GPIO42: IC1.35 (IO42), J4.8 (Pin_8)
- new net GPIO45: IC1.26 (IO45), J4.14 (Pin_14)
- new net GPIO46: IC1.16 (IO46), J3.14 (Pin_14)
- new net GPIO47: IC1.24 (IO47), J4.16 (Pin_16)
- new net GPIO48: IC1.25 (IO48), J4.15 (Pin_15)
- new net GPIO5_CS: IC1.5 (IO5), J2.2 (CD/DAT3), J3.3 (Pin_3)
- new net GPIO6: IC1.6 (IO6), J3.4 (Pin_4)
- new net GPIO7: IC1.7 (IO7), J3.5 (Pin_5)
- new net GPIO8: IC1.12 (IO8), J3.10 (Pin_10)
- new net GPIO9: IC1.17 (IO9), J3.15 (Pin_15)
- new net SCL: HM1.4 (SCK), IC1.10 (IO17), IC3.7 (SCL), IC5.18 (B2), J3.8 (Pin_8), J8.1 (Pin_1), R22.1
- new net SCL_low: IC5.3 (A2), IC7.23 (SCL_/_SCLK)
- new net SDA: HM1.3 (SDI), IC1.9 (IO16), IC3.8 (SDA), IC5.17 (B3), J3.7 (Pin_7), J8.2 (Pin_2), R21.1
- new net SDA_low: IC5.4 (A3), IC7.24 (SDA_/_SDI)
- no-connect marks 0 -> 57
Other:
- note added: "1.8V Voltage Regulator"
- note added: "3.3V Converter"
- note added: "Auto-Reset"
- note added: "BME280"
- note added: "Connect to enable LiPo Battery"
- note added: "Debug Serial"
- note added: "Debug USB"
- note added: "ESP32"
- note added: "Fuel Gauge"
- note added: "I2C"
- note added: "I2C Level Shifter"
- note added: "ICM-20948"
- note added: "IO Headers"
- note added: "LiPo Manager"
- note added: "Passt die Diode? Funktion: USB angeschlossen => Batterie lädt USB nicht angeschlossen => Batterie versorgt Spannungswandler"
- note added: "SD-Card-Module"
- note added: "USB C"
- note added: "USB to Serial"
- note added: "Use to set i2c adresse"
- note added: "Use to set i2c adresse 1-2: 0x118 2-3: 0x119"
